Commit message: Gazebo stuff added

File: description/robot_core.xacro (robot description, xacro)
@@ -30,4 +30,7 @@
         <origin xyz="0 0 0"/>
     </joint>
+    <gazebo reference="body_link">
+        <material>Gazebo/Orange</material>
+    </gazebo>
     <!-- WHEELS -->
     <!-- LEFT WHEEL -->
@@ -51,7 +54,10 @@
         <parent link="base_link"/>
         <child link="wheel_left_link"/>
-        <origin xyz="0 0.06025 0" rpy="-${pi/2} 0 0"/>
+        <origin xyz="0 0.0685 0" rpy="-${pi/2} 0 0"/>
         <axis xyz="0 0 1"/>
     </joint>
+    <gazebo reference="wheel_left_link">
+        <material>Gazebo/Blue</material>
+    </gazebo>
     <!-- RIGHT WHEEL -->
     <link name="wheel_right_link">
@@ -74,7 +80,10 @@
         <parent link="base_link"/>
         <child link="wheel_right_link"/>
-        <origin xyz="0 -0.06025 0" rpy="${pi/2} 0 0"/>
+        <origin xyz="0 -0.0685 0" rpy="${pi/2} 0 0"/>
         <axis xyz="0 0 -1"/>
     </joint>
+    <gazebo reference="wheel_right_link">
+        <material>Gazebo/Blue</material>
+    </gazebo>
     <!-- CASTER WHEELS-->
     <!-- RIGHT FRONT CASTER-->
@@ -99,4 +108,9 @@
         <origin xyz="0.08435 -0.0431 -0.01875"/>
     </joint>
+    <gazebo reference="caster_rf_link">
+        <material>Gazebo/Orange</material>
+        <mu1 value="0.001"/>
+        <mu2 value="0.001"/>
+    </gazebo>
     <!-- LEFT FRONT CASTER-->
     <link name="caster_lf_link">
@@ -121,4 +135,9 @@
         <origin xyz="0.08435 0.0431 -0.01875"/>
     </joint>
+    <gazebo reference="caster_lf_link">
+        <material>Gazebo/Orange</material>
+        <mu1 value="0.001"/>
+        <mu2 value="0.001"/>
+    </gazebo>
     <!-- RIGHT REAR CASTER-->
     <link name="caster_rr_link">
@@ -143,4 +162,9 @@
         <origin xyz="-0.08435 -0.0431 -0.01875"/>
     </joint>
+    <gazebo reference="caster_rr_link">
+        <material>Gazebo/Orange</material>
+        <mu1 value="0.001"/>
+        <mu2 value="0.001"/>
+    </gazebo>
     <!-- LEFT REAR CASTER-->
     <link name="caster_lr_link">
@@ -165,3 +189,8 @@
         <origin xyz="-0.08435 0.0431 -0.01875"/>
     </joint>
+    <gazebo reference="caster_lr_link">
+        <material>Gazebo/Orange</material>
+        <mu1 value="0.001"/>
+        <mu21 value="0.001"/>
+    </gazebo>
 </robot>

Commit message: Lidar added

File: description/robot_core.xacro (robot description, xacro)
@@ -9,18 +9,18 @@
     <link name="body_link">
         <visual>
-            <origin xyz="0 0 0.0665"/>
-            <geometry>
-                <box size="0.2 0.179 0.154"/>
-            </geometry>
-            <material name="orange"/>
-        </visual>
-        <collision>
-            <origin xyz="0 0 0.0665"/>
-            <geometry>
-                <box size="0.2 0.179 0.154"/>
-            </geometry>
-        </collision>
-        <xacro:inertial_box mass="2" x="0.2" y="0.179" z="0.154">
-            <origin xyz="0 0 0.0665"/>
+            <origin xyz="0 0 0.04875"/>
+            <geometry>
+                <box size="0.2 0.1795 0.1185"/>
+            </geometry>
+            <material name="orange"/>
+        </visual>
+        <collision>
+            <origin xyz="0 0 0.04875"/>
+            <geometry>
+                <box size="0.2 0.1795 0.1185"/>
+            </geometry>
+        </collision>
+        <xacro:inertial_box mass="2" x="0.2" y="0.1795" z="0.1185">
+            <origin xyz="0 0 0.04875"/>
         </xacro:inertial_box>
     </link>
@@ -33,4 +33,83 @@
         <material>Gazebo/Orange</material>
     </gazebo>
+    <!-- COLUMNS -->
+    <link name="columns_link">
+        <!-- FRONT RIGHT -->
+        <visual>
+            <origin xyz="0.093306 -0.07725 0"/>
+            <geometry>
+                <box size="0.015 0.025 0.030"/>
+            </geometry>
+            <material name="orange"/>
+        </visual>
+        <!-- FRONT LEFT -->
+        <visual>
+            <origin xyz="0.088306 0.08225 0"/>
+            <geometry>
+                <box size="0.025 0.015 0.030"/>
+            </geometry>
+            <material name="orange"/>
+        </visual>
+        <!-- REAR RIGHT -->
+        <visual>
+            <origin xyz="-0.088306 -0.08225 0"/>
+            <geometry>
+                <box size="0.025 0.015 0.030"/>
+            </geometry>
+            <material name="orange"/>
+        </visual>
+        <!-- REAR LEFT -->
+        <visual>
+            <origin xyz="-0.093306 0.07725 0"/>
+            <geometry>
+                <box size="0.015 0.025 0.030"/>
+            </geometry>
+            <material name="orange"/>
+        </visual>
+        <collision>
+            <origin xyz="0 0 0.0"/>
+            <geometry>
+                <box size="0.2 0.1795 0.030"/>
+            </geometry>
+        </collision>
+        <xacro:inertial_box mass="0.001" x="0.2" y="0.1795" z="0.030">
+            <origin xyz="0 0 0.0"/>
+        </xacro:inertial_box>
+    </link>
+    <joint name="columns_joint" type="fixed">
+        <parent link="body_link"/>
+        <child link="columns_link"/>
+        <origin xyz="0 0 0.123"/>
+    </joint>
+    <gazebo reference="columns_link">
+        <material>Gazebo/Orange</material>
+    </gazebo>
+    <!-- PLATFORM -->
+    <link name="platform_link">
+        <visual>
+            <origin xyz="0 0 0"/>
+            <geometry>
+                <box size="0.2 0.1795 0.006"/>
+            </geometry>
+            <material name="orange"/>
+        </visual>
+        <collision>
+            <origin xyz="0 0 0"/>
+            <geometry>
+                <box size="0.2 0.1795 0.006"/>
+            </geometry>
+        </collision>
+        <xacro:inertial_box mass="0.001" x="0.2" y="0.1795" z="0.006">
+            <origin xyz="0 0 00"/>
+        </xacro:inertial_box>
+    </link>
+    <joint name="platform_joint" type="fixed">
+        <parent link="body_link"/>
+        <child link="platform_link"/>
+        <origin xyz="0 0 0.141"/>
+    </joint>
+    <gazebo reference="platform_link">
+        <material>Gazebo/Orange</material>
+    </gazebo>
     <!-- WHEELS -->
     <!-- LEFT WHEEL -->
@@ -38,5 +117,5 @@
         <visual>
             <geometry>
-                <cylinder radius="0.0255" length="0.015"/>
+                <cylinder radius="0.026" length="0.015"/>
             </geometry>
             <material name="blue"/>
@@ -44,9 +123,9 @@
         <collision>
             <geometry>
-                <cylinder radius="0.0255" length="0.015"/>
-            </geometry>
-        </collision>
-        <xacro:inertial_cylinder mass="0.1" length="0.015" radius="0.0255">
-            <origin xyz="0 0 0"/>
+                <cylinder radius="0.026" length="0.015"/>
+            </geometry>
+        </collision>
+        <xacro:inertial_cylinder mass="0.1" length="0.015" radius="0.026">
+            <origin xyz="0 0 0" rpy="0 0 0"/>
         </xacro:inertial_cylinder>
     </link>
@@ -54,5 +133,5 @@
         <parent link="base_link"/>
         <child link="wheel_left_link"/>
-        <origin xyz="0 0.0685 0" rpy="-${pi/2} 0 0"/>
+        <origin xyz="0 0.07225 0" rpy="-${pi/2} 0 0"/>
         <axis xyz="0 0 1"/>
     </joint>
@@ -64,5 +143,5 @@
         <visual>
             <geometry>
-                <cylinder radius="0.0255" length="0.015"/>
+                <cylinder radius="0.026" length="0.015"/>
             </geometry>
             <material name="blue"/>
@@ -70,9 +149,9 @@
         <collision>
             <geometry>
-                <cylinder radius="0.0255" length="0.015"/>
-            </geometry>
-        </collision>
-        <xacro:inertial_cylinder mass="0.1" length="0.015" radius="0.0255">
-            <origin xyz="0 0 0"/>
+                <cylinder radius="0.026" length="0.015"/>
+            </geometry>
+        </collision>
+        <xacro:inertial_cylinder mass="0.1" length="0.015" radius="0.026">
+            <origin xyz="0 0 0" rpy="0 0 0"/>
         </xacro:inertial_cylinder>
     </link>
@@ -80,8 +159,8 @@
         <parent link="base_link"/>
         <child link="wheel_right_link"/>
-        <origin xyz="0 -0.0685 0" rpy="${pi/2} 0 0"/>
+        <origin xyz="0 -0.07225 0" rpy="${pi/2} 0 0"/>
         <axis xyz="0 0 -1"/>
     </joint>
-    <gazebo reference="wheel_right_link">
+     <gazebo reference="wheel_left_link">
         <material>Gazebo/Blue</material>
     </gazebo>
@@ -91,13 +170,13 @@
         <visual>
             <geometry>
-                <sphere radius="0.00675"/>
-            </geometry>
-        </visual>
-        <collision>
-            <geometry>
-                <sphere radius="0.00675"/>
-            </geometry>
-        </collision>
-        <xacro:inertial_sphere mass="0.01" radius="0.00675">
+                <sphere radius="0.00625"/>
+            </geometry>
+        </visual>
+        <collision>
+            <geometry>
+                <sphere radius="0.00625"/>
+            </geometry>
+        </collision>
+        <xacro:inertial_sphere mass="0.01" radius="0.00625">
             <origin xyz="0 0 0"/>
         </xacro:inertial_sphere>
@@ -106,5 +185,5 @@
         <parent link="body_link"/>
         <child link="caster_rf_link"/>
-        <origin xyz="0.08435 -0.0431 -0.01875"/>
+        <origin xyz="0.08435 -0.0431 -0.01825"/>
     </joint>
     <gazebo reference="caster_rf_link">
@@ -117,14 +196,14 @@
         <visual>
             <geometry>
-                <sphere radius="0.00675"/>
-            </geometry>
-            <material name="orange"/>
-        </visual>
-        <collision>
-            <geometry>
-                <sphere radius="0.00675"/>
-            </geometry>
-        </collision>
-        <xacro:inertial_sphere mass="0.01" radius="0.00675">
+                <sphere radius="0.00625"/>
+            </geometry>
+            <material name="orange"/>
+        </visual>
+        <collision>
+            <geometry>
+                <sphere radius="0.00625"/>
+            </geometry>
+        </collision>
+        <xacro:inertial_sphere mass="0.01" radius="0.00625">
             <origin xyz="0 0 0"/>
         </xacro:inertial_sphere>
@@ -133,5 +212,5 @@
         <parent link="body_link"/>
         <child link="caster_lf_link"/>
-        <origin xyz="0.08435 0.0431 -0.01875"/>
+        <origin xyz="0.08435 0.0431 -0.01825"/>
     </joint>
     <gazebo reference="caster_lf_link">
@@ -144,14 +223,14 @@
         <visual>
             <geometry>
-                <sphere radius="0.00675"/>
-            </geometry>
-            <material name="orange"/>
-        </visual>
-        <collision>
-            <geometry>
-                <sphere radius="0.00675"/>
-            </geometry>
-        </collision>
-        <xacro:inertial_sphere mass="0.01" radius="0.00675">
+                <sphere radius="0.00625"/>
+            </geometry>
+            <material name="orange"/>
+        </visual>
+        <collision>
+            <geometry>
+                <sphere radius="0.00625"/>
+            </geometry>
+        </collision>
+        <xacro:inertial_sphere mass="0.01" radius="0.00625">
             <origin xyz="0 0 0"/>
         </xacro:inertial_sphere>
@@ -160,5 +239,5 @@
         <parent link="body_link"/>
         <child link="caster_rr_link"/>
-        <origin xyz="-0.08435 -0.0431 -0.01875"/>
+        <origin xyz="-0.08435 -0.0431 -0.01825"/>
     </joint>
     <gazebo reference="caster_rr_link">
@@ -171,14 +250,14 @@
         <visual>
             <geometry>
-                <sphere radius="0.00675"/>
-            </geometry>
-            <material name="orange"/>
-        </visual>
-        <collision>
-            <geometry>
-                <sphere radius="0.00675"/>
-            </geometry>
-        </collision>
-        <xacro:inertial_sphere mass="0.01" radius="0.00675">
+                <sphere radius="0.00625"/>
+            </geometry>
+            <material name="orange"/>
+        </visual>
+        <collision>
+            <geometry>
+                <sphere radius="0.00625"/>
+            </geometry>
+        </collision>
+        <xacro:inertial_sphere mass="0.01" radius="0.00625">
             <origin xyz="0 0 0"/>
         </xacro:inertial_sphere>
@@ -187,5 +266,5 @@
         <parent link="body_link"/>
         <child link="caster_lr_link"/>
-        <origin xyz="-0.08435 0.0431 -0.01875"/>
+        <origin xyz="-0.08435 0.0431 -0.01825"/>
     </joint>
     <gazebo reference="caster_lr_link">

Commit message: SLAM

File: description/robot_core.xacro (robot description, xacro)
@@ -6,4 +6,12 @@
     <link name="base_link">
     </link>
+    <!-- BASE FOOTPRINT -->
+    <link name="base_footprint">
+    </link>
+    <joint name="base_footprint_joint" type="fixed">
+        <parent link="base_link"/>
+        <child link="base_footprint"/>
+        <origin xyz="0 0 0" rpy="0 0 0"/>
+    </joint>
     <!-- BODY -->
     <link name="body_link">
