Commit message: navigation

File: description/lidar.xacro (robot description, xacro)
@@ -2,7 +2,9 @@
 <robot xmlns:xacro="http://www.ros.org/wiki/xacro" >
     <joint name="laser_joint" type="fixed">
-        <parent link="body_link"/>
+        <!-- <parent link="body_link"/>-->
+        <parent link="base_link"/>
         <child link="laser_frame"/>
-        <origin xyz="0 0 0.117" rpy="0 0 0"/>
+        <origin xyz="0 0 0.16575" rpy="0 0 0"/>
+        <!--<origin xyz="0 0 0.117" rpy="0 0 0"/>-->
     </joint>
     <link name="laser_frame">
@@ -11,5 +13,5 @@
                 <cylinder radius="0.0355" length="0.0185"/>
             </geometry>
-            <material name="red"/>
+            <material name="black"/>
         </visual>
         <collision>
